File: src/kicad/newParts.sch (KiCad schematic (older format))
At the start: 3 parts, among them U2 74HC08, U3 74HC4511D, U4 HEF4518BT

Commit message: added basic circuit layout
Parts:
- added U12, U2E1, U8: 74HC08, Housings_SOIC:SOIC-14_3.9x8.7mm_Pitch1.27mm, symbol PB170:74HC08
Changed lines of the file:
@@
 $Descr A4 11693 8268
 encoding utf-8
-Sheet 2 2
+Sheet 1 2
 Title ""
 Date ""
@@
 	1    0    0    -1
 $EndComp
+$Comp
+L PB170:74HC08 U8
+U 4 1 5FF686CD
+P 1800 1950
+F 0 "U8" H 1825 2217 50  0000 C CNN
+F 1 "74HC08" H 1825 2126 50  0000 C CNN
+F 2 "Housings_SOIC:SOIC-14_3.9x8.7mm_Pitch1.27mm" H 1800 1950 50  0001 C CNN
+F 3 "https://datasheet.lcsc.com/szlcsc/Nexperia-74HC08D-653_C5593.pdf" H 1800 1950 50  0001 C CNN
+F 4 "C5593" H 1800 1950 50  0001 C CNN "LCSC"
+	4    1800 1950
+	1    0    0    -1
+$EndComp
+$Comp
+L PB170:74HC08 U12
+U 1 1 5FF686D4
+P 2550 1950
+F 0 "U12" H 2575 2217 50  0000 C CNN
+F 1 "74HC08" H 2575 2126 50  0000 C CNN
+F 2 "Housings_SOIC:SOIC-14_3.9x8.7mm_Pitch1.27mm" H 2550 1950 50  0001 C CNN
+F 3 "https://datasheet.lcsc.com/szlcsc/Nexperia-74HC08D-653_C5593.pdf" H 2550 1950 50  0001 C CNN
+F 4 "C5593" H 2550 1950 50  0001 C CNN "LCSC"
+	1    2550 1950
+	1    0    0    -1
+$EndComp
+$Comp
+L PB170:74HC08 U12
+U 3 1 5FF686DB
+P 3300 1950
+F 0 "U12" H 3325 2217 50  0000 C CNN
+F 1 "74HC08" H 3325 2126 50  0000 C CNN
+F 2 "Housings_SOIC:SOIC-14_3.9x8.7mm_Pitch1.27mm" H 3300 1950 50  0001 C CNN
+F 3 "https://datasheet.lcsc.com/szlcsc/Nexperia-74HC08D-653_C5593.pdf" H 3300 1950 50  0001 C CNN
+F 4 "C5593" H 3300 1950 50  0001 C CNN "LCSC"
+	3    3300 1950
+	1    0    0    -1
+$EndComp
+$Comp
+L PB170:74HC08 U8
+U 3 1 5FF6C8B4
+P 1000 2450
+F 0 "U8" H 1025 2717 50  0000 C CNN
+F 1 "74HC08" H 1025 2626 50  0000 C CNN
+F 2 "Housings_SOIC:SOIC-14_3.9x8.7mm_Pitch1.27mm" H 1000 2450 50  0001 C CNN
+F 3 "https://datasheet.lcsc.com/szlcsc/Nexperia-74HC08D-653_C5593.pdf" H 1000 2450 50  0001 C CNN
+F 4 "C5593" H 1000 2450 50  0001 C CNN "LCSC"
+	3    1000 2450
+	1    0    0    -1
+$EndComp
+$Comp
+L PB170:74HC08 U8
+U 5 1 5FF6C8BB
+P 1800 2450
+F 0 "U8" H 1825 2717 50  0000 C CNN
+F 1 "74HC08" H 1825 2626 50  0000 C CNN
+F 2 "Housings_SOIC:SOIC-14_3.9x8.7mm_Pitch1.27mm" H 1800 2450 50  0001 C CNN
+F 3 "https://datasheet.lcsc.com/szlcsc/Nexperia-74HC08D-653_C5593.pdf" H 1800 2450 50  0001 C CNN
+F 4 "C5593" H 1800 2450 50  0001 C CNN "LCSC"
+	5    1800 2450
+	1    0    0    -1
+$EndComp
+$Comp
+L PB170:74HC08 U12
+U 2 1 5FF6C8C2
+P 2550 2450
+F 0 "U12" H 2575 2717 50  0000 C CNN
+F 1 "74HC08" H 2575 2626 50  0000 C CNN
+F 2 "Housings_SOIC:SOIC-14_3.9x8.7mm_Pitch1.27mm" H 2550 2450 50  0001 C CNN
+F 3 "https://datasheet.lcsc.com/szlcsc/Nexperia-74HC08D-653_C5593.pdf" H 2550 2450 50  0001 C CNN
+F 4 "C5593" H 2550 2450 50  0001 C CNN "LCSC"
+	2    2550 2450
+	1    0    0    -1
+$EndComp
+$Comp
+L PB170:74HC08 U12
+U 4 1 5FF6C8C9
+P 3300 2450
+F 0 "U12" H 3325 2717 50  0000 C CNN
+F 1 "74HC08" H 3325 2626 50  0000 C CNN
+F 2 "Housings_SOIC:SOIC-14_3.9x8.7mm_Pitch1.27mm" H 3300 2450 50  0001 C CNN
+F 3 "https://datasheet.lcsc.com/szlcsc/Nexperia-74HC08D-653_C5593.pdf" H 3300 2450 50  0001 C CNN
+F 4 "C5593" H 3300 2450 50  0001 C CNN "LCSC"
+	4    3300 2450
+	1    0    0    -1
+$EndComp
+$Comp
+L PB170:74HC08 U2E1
+U 1 1 5FF686C6
+P 1000 1950
+F 0 "U2E1" H 1025 2217 50  0000 C CNN
+F 1 "74HC08" H 1025 2126 50  0000 C CNN
+F 2 "Housings_SOIC:SOIC-14_3.9x8.7mm_Pitch1.27mm" H 1000 1950 50  0001 C CNN
+F 3 "https://datasheet.lcsc.com/szlcsc/Nexperia-74HC08D-653_C5593.pdf" H 1000 1950 50  0001 C CNN
+F 4 "C5593" H 1000 1950 50  0001 C CNN "LCSC"
+	1    1000 1950
+	1    0    0    -1
+$EndComp
